File: main/main.kicad_sch (KiCad schematic)
At the start: 9 parts

Commit message: imu
Parts:
- removed BSC1: C, Library:res0603, symbol Device:C
- removed BSC2: 1n5, Library:cap0603, symbol Device:C
- removed BSD1: 1N5401, Diode_THT:D_DO-201AD_P15.24mm_Horizontal, symbol Diode:1N5401
- removed BSJ1: XT30, Library:xt30-f, symbol Connector_Generic:Conn_01x02
- removed BSQ1: IRLB3036PbF, Library:TO-220-3_Vertical, symbol vincent:IPD050N10N5ATMA1
- removed BSR1: 20R, Library:res0603, symbol Device:R
- removed BSR2, BSR3: R, Library:res0603, symbol Device:R
- removed BSU1: NCP81074AMNTBG, Library:SON50P200X200X100-9N, symbol senrobo_kicad:NCP81074XMNTBG
Other:
- added sheet boost (boost.kicad_sch)
- added sheet imu (imu.kicad_sch)
