File: main/boost.kicad_sch (KiCad schematic)
At the start: 9 parts

Commit message: cooked up a pcb layout
Parts:
- added J3: Conn_01x01_Pin, Connector_PinHeader_2.54mm:PinHeader_1x01_P2.54mm_Vertical, symbol Connector:Conn_01x01_Pin
- BSC1: value C -> 0.1u
- BSR2, BSR3: value R -> 100
Connections:
- net Sol: now also J3.1 (Pin_1)
Other:
- note added: "keep traces short and wide"
- note added: "put decoup caps as close to gate drive IC"
- note added: "put driver as close to mosfet as possible"
Changed lines of the file:
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@@
 		(color 0 0 0 0)
 	)
+	(junction
+		(at 107.95 96.52)
+		(diameter 0)
+		(color 0 0 0 0)
+	)
 	(wire
 		(pts
@@
 	(wire
 		(pts
+			(xy 102.87 91.44) (xy 107.95 91.44)
+		)
+		(stroke
+			(width 0)
+			(type default)
+		)
+	)
+	(wire
+		(pts
 			(xy 148.59 104.14) (xy 148.59 111.76)
 		)
@@
 	(wire
 		(pts
+			(xy 107.95 91.44) (xy 107.95 96.52)
+		)
+		(stroke
+			(width 0)
+			(type default)
+		)
+	)
+	(wire
+		(pts
 			(xy 148.59 111.76) (xy 166.37 111.76)
 		)
@@
 			(width 0)
 			(type default)
+		)
+	)
+	(text "put decoup caps as close to gate drive IC"
+		(exclude_from_sim no)
+		(at 198.628 85.344 0)
+		(effects
+			(font
+				(size 1.27 1.27)
+			)
+		)
+	)
+	(text "put driver as close to mosfet as possible\n"
+		(exclude_from_sim no)
+		(at 198.12 81.788 0)
+		(effects
+			(font
+				(size 1.27 1.27)
+			)
+		)
+	)
+	(text "keep traces short and wide"
+		(exclude_from_sim no)
+		(at 191.008 83.82 0)
+		(effects
+			(font
+				(size 1.27 1.27)
+			)
 		)
 	)
@@
 			)
 		)
-		(property "Value" "R"
+		(property "Value" "100"
 			(at 132.08 101.6 90)
 			(effects
@@
 			)
 		)
-		(property "Value" "R"
+		(property "Value" "100"
 			(at 132.08 96.52 90)
 			(effects
@@
 				(path "/55c0a6b2-6fc9-44ca-8d10-659d11d090d5/e2785760-ff03-4094-8a17-cb2995826734"
 					(reference "BSR2")
+					(unit 1)
+				)
+			)
+		)
+	)
+	(symbol
+		(lib_id "Connector:Conn_01x01_Pin")
+		(at 97.79 91.44 0)
+		(unit 1)
+		(exclude_from_sim no)
+		(in_bom yes)
+		(on_board yes)
+		(dnp no)
+		(fields_autoplaced yes)
+		(property "Reference" "J3"
+			(at 98.425 86.36 0)
+			(effects
+				(font
+					(size 1.27 1.27)
+				)
+			)
+		)
+		(property "Value" "Conn_01x01_Pin"
+			(at 98.425 88.9 0)
+			(effects
+				(font
+					(size 1.27 1.27)
+				)
+			)
+		)
+		(property "Footprint" "Connector_PinHeader_2.54mm:PinHeader_1x01_P2.54mm_Vertical"
+			(at 97.79 91.44 0)
+			(effects
+				(font
+					(size 1.27 1.27)
+				)
+				(hide yes)
+			)
+		)
+		(property "Datasheet" "~"
+			(at 97.79 91.44 0)
+			(effects
+				(font
+					(size 1.27 1.27)
+				)
+				(hide yes)
+			)
+		)
+		(property "Description" "Generic connector, single row, 01x01, script generated"
+			(at 97.79 91.44 0)
+			(effects
+				(font
+					(size 1.27 1.27)
+				)
+				(hide yes)
+			)
+		)
+		(pin "1"
+		)
+		(instances
+			(project ""
+				(path "/55c0a6b2-6fc9-44ca-8d10-659d11d090d5/e2785760-ff03-4094-8a17-cb2995826734"
+					(reference "J3")
 					(unit 1)
 				)
@@
 			)
 		)
-		(property "Value" "C"
+		(property "Value" "0.1u"
 			(at 137.16 78.7399 0)
 			(effects
