File: main/imu.kicad_sch (KiCad schematic)
At the start: 25 parts, among them IC1 ICM-42688-P, J1 Conn_01x06, J2 Conn_01x04, U1 STM32G071GBUx, U2 16MHz

Commit message: cooked up a pcb layout
Parts:
- J1: footprint (none) -> Connector_PinHeader_2.54mm:PinHeader_1x06_P2.54mm_Vertical
Changed lines of the file:
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@@
 			)
 		)
-		(property "Footprint" ""
+		(property "Footprint" "Connector_PinHeader_2.54mm:PinHeader_1x06_P2.54mm_Vertical"
 			(at 195.58 35.56 0)
 			(effects
