File: main/main.kicad_pcb (KiCad board)
At the start: 2 copper layers, 9 parts

Commit message: imu
Parts:
- added C1: 2u2, Library:cap0603, F.Cu at (117.4, 59.1)
- added C10: 10p, Capacitor_SMD:C_0402_1005Metric_Pad0.74x0.62mm_HandSolder, F.Cu at (113.4, 72.3)
- added C2: 2u2, Library:cap0603, F.Cu at (117.4, 62.2)
- added C3: 2u2, Capacitor_SMD:C_0402_1005Metric_Pad0.74x0.62mm_HandSolder, F.Cu at (113.4, 58.5)
- added C4: 0u1, Capacitor_SMD:C_0402_1005Metric_Pad0.74x0.62mm_HandSolder, F.Cu at (113.4, 60.5)
- added C5: 0u1, Capacitor_SMD:C_0402_1005Metric_Pad0.74x0.62mm_HandSolder, F.Cu at (113.4, 62.4)
- added C6: 2u2, Capacitor_SMD:C_0402_1005Metric_Pad0.74x0.62mm_HandSolder, F.Cu at (113.4, 64.4)
- added C7: 10n, Capacitor_SMD:C_0402_1005Metric_Pad0.74x0.62mm_HandSolder, F.Cu at (113.4, 66.4)
- added C8: 0u1, Capacitor_SMD:C_0402_1005Metric_Pad0.74x0.62mm_HandSolder, F.Cu at (113.4, 68.3)
- added C9: 10p, Capacitor_SMD:C_0402_1005Metric_Pad0.74x0.62mm_HandSolder, F.Cu at (113.4, 70.3)
- added D1: RCLAMP0521PATCT, Library:RCLAMP0521PATCT, F.Cu at (110.1, 58.9)
- added D2: RCLAMP0521PATCT, Library:RCLAMP0521PATCT, F.Cu at (110.1, 61.6)
- added D3: RCLAMP0521PATCT, Library:RCLAMP0521PATCT, F.Cu at (110.1, 64.3)
- added D4: RCLAMP0521PATCT, Library:RCLAMP0521PATCT, F.Cu at (110.1, 67.0)
- added D5: RCLAMP0521PATCT, Library:RCLAMP0521PATCT, F.Cu at (110.1, 69.7)
- added D6: RCLAMP0521PATCT, Library:RCLAMP0521PATCT, F.Cu at (110.1, 72.4)
- added D7: RED, Library:led0603, F.Cu at (117.4, 65.3)
- added FB1: 100R, Library:fb0603, F.Cu at (117.4, 68.4)
- added IC1: ICM-42688-P, Library:IIM42352, F.Cu at (122.1, 73.1)
- added J2: Conn_01x04, Connector_PinHeader_2.54mm:PinHeader_2x02_P2.54mm_Vertical, F.Cu at (122.1, 59.8)
- added R1: 1K, Resistor_SMD:R_0402_1005Metric, F.Cu at (125.9, 72.0)
- added R2: R, Resistor_SMD:R_0402_1005Metric, F.Cu at (125.9, 74.0)
- added U1: STM32G071GBUx, Package_DFN_QFN:QFN-28_4x4mm_P0.5mm, F.Cu at (122.9, 67.9)
- added U2: 16MHz, Library:830108288709, F.Cu at (117.4, 72.0)

Commit message: cooked up a pcb layout
Parts:
- added J1: Conn_01x06, Connector_PinHeader_2.54mm:PinHeader_1x06_P2.54mm_Vertical, F.Cu at (16.5, 72.8)
- added J3: Conn_01x01_Pin, Connector_PinHeader_2.54mm:PinHeader_1x01_P2.54mm_Vertical, F.Cu at (38.9, 37.8)
- BSC1: value C -> 0.1u
- BSR2, BSR3: value R -> 100
- moved J2 103.0 mm to (19.1, 56.4), turned to 180 degrees
- moved C1 95.2 mm to (22.4, 53.8), turned to 90 degrees
- moved FB1 94.6 mm to (23.5, 56.8)
- moved C2 93.3 mm to (24.5, 53.8), turned to 90 degrees
- moved R1 92.7 mm to (33.2, 72.8), turned to 180 degrees
- moved U1 91.8 mm to (31.1, 67.0)
- moved U2 91.0 mm to (26.6, 65.8), turned to 90 degrees
- moved R2 90.6 mm to (35.8, 64.8), turned to 180 degrees
- moved C10 89.9 mm to (23.7, 66.5), turned to 180 degrees
- moved C9 89.9 mm to (23.7, 65.2), turned to 180 degrees
- moved IC1 88.9 mm to (34.1, 60.1), turned to 180 degrees
- moved C3 87.0 mm to (27.1, 69.6), turned to 180 degrees
- moved C4 86.7 mm to (27.1, 68.5), turned to 180 degrees
- moved D7 84.4 mm to (33.2, 71.0), turned to 180 degrees
- moved D1 83.2 mm to (27.9, 71.5), turned to -90 degrees
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Routing:
- net /imu/MCU1 SWDIO: track 0.00 -> 37.8 mm, vias 0 -> 3
- net +3V3 FILT: track 0.00 -> 35.2 mm, vias 0 -> 2
- net /imu/MCU1 SWCLK: track 0.00 -> 31.3 mm, vias 0 -> 1
- net +3V3: track 0.00 -> 23.5 mm
- net Net-(BSD1-A): track 0.00 -> 20.3 mm
- net /imu/UART RX: track 0.00 -> 19.5 mm, vias 0 -> 2
- net /imu/MPU SCL: track 0.00 -> 18.0 mm, vias 0 -> 2
- net /imu/UART TX: track 0.00 -> 15.7 mm
- net /imu/MPU SDA: track 0.00 -> 14.1 mm
- net /imu/MPU MOSI: track 0.00 -> 11.4 mm, vias 0 -> 2
- net /imu/MPU MISO: track 0.00 -> 8.19 mm, vias 0 -> 2
- net Net-(BSQ1-G): track 0.00 -> 6.65 mm
- net /imu/MCU1 OSC OUT: track 0.00 -> 6.56 mm
- net /imu/MCU1 OSC IN: track 0.00 -> 5.85 mm
- net /imu/MPU CS: track 0.00 -> 5.29 mm
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- added copper zone on F.Cu, net +12V
- added copper zone on F.Cu, net +48V
- added copper zone on B.Cu, net GND
- added copper zone on B.Cu, net GNDREF
- added copper zone on F.Cu, net GNDREF
Other:
- board text added: "3v3"
- board text added: "gnd"
- board text added: "rx"
- board text added: "scl"
- board text added: "sda"
- board text added: "sol"
- board text added: "swclk"
- board text added: "swdio"
- board text added: "tx"
